Commit message: open gripper, and move

File: src/indy7_ign-main/urdf/indy7.urdf (robot description, URDF)
Before this commit: robot indy7, 11 links, 10 joints
Joints:
- joint end_effector_frame_fixed_joint: parent indy7_link6 -> indy7_hand
- joint indy7_hand_joint: origin xyz=0 0 0.107 rpy=0 0 -0.7853981633974483 -> xyz=0 0 0.064 rpy=0 0 -0.7853981633974483
